File: RP2350A_Dev_board/RP2350A_Dev_board.kicad_pcb (KiCad board)
At the start: 2 copper layers, 74.7 x 64.3 mm, 3 parts, among them U1 W25Q128JVP

Commit message: почти всё, осталось только шелкографию сделать и готово
Parts:
- added C1: 10uF, Capacitor_SMD:C_0603_1608Metric, F.Cu at (116.2, 95.8)
- added C10: 100nF, Capacitor_SMD:C_0603_1608Metric, F.Cu at (112.5, 81.2)
- added C11: 10pF, Capacitor_SMD:C_0603_1608Metric, F.Cu at (125.5, 76.5)
- added C12: 100nF, Capacitor_SMD:C_0603_1608Metric, F.Cu at (111.7, 85.3)
- added C13: 10uF, Capacitor_SMD:C_0603_1608Metric, F.Cu at (111.0, 93.0)
- added C14: 100nF, Capacitor_SMD:C_0603_1608Metric, F.Cu at (112.5, 90.0)
- added C15: 20pF, Capacitor_SMD:C_0603_1608Metric, F.Cu at (115.9, 76.9)
- added C16: 100nF, Capacitor_SMD:C_0603_1608Metric, F.Cu at (123.9, 93.5)
- added C17: 22uF, Capacitor_SMD:C_0402_1005Metric, F.Cu at (118.7, 114.6)
- added C18: 22uF, Capacitor_SMD:C_0402_1005Metric, F.Cu at (119.8, 118.4)
- added C19: 100nF, Capacitor_SMD:C_0402_1005Metric, F.Cu at (119.8, 117.5)
- added C2: 20pF, Capacitor_SMD:C_0603_1608Metric, F.Cu at (121.6, 76.8)
- added C20: 100nF, Capacitor_SMD:C_0402_1005Metric, F.Cu at (117.2, 111.8)
- added C21: 100nF, Capacitor_SMD:C_0402_1005Metric, F.Cu at (115.7, 112.7)
- added C22: 22uF, Capacitor_SMD:C_0402_1005Metric, F.Cu at (119.8, 119.3)
- added C23: 22uF, Capacitor_SMD:C_0402_1005Metric, F.Cu at (115.7, 111.0)
- added C3: 10pF, Capacitor_SMD:C_0603_1608Metric, F.Cu at (111.7, 86.8)
- added C4: 100nF, Capacitor_SMD:C_0603_1608Metric, F.Cu at (127.0, 86.7)
- added C5: 100nF, Capacitor_SMD:C_0603_1608Metric, F.Cu at (127.0, 84.3)
- added C6: 10pF, Capacitor_SMD:C_0603_1608Metric, F.Cu at (124.5, 78.9)
- added C7: 100nF, Capacitor_SMD:C_0603_1608Metric, F.Cu at (111.0, 91.5)
- added C8: 10uF, Capacitor_SMD:C_0603_1608Metric, F.Cu at (118.8, 93.6)
- added C9: 10uF, Capacitor_SMD:C_0603_1608Metric, F.Cu at (114.7, 95.8)
- added D1: LED, LED_SMD:LED_0603_1608Metric, F.Cu at (102.2, 101.1)
- added D2: LED, LED_SMD:LED_0603_1608Metric, F.Cu at (102.2, 102.9)
- added D3: LED, LED_SMD:LED_0603_1608Metric, F.Cu at (102.2, 104.6)
- added DD5: ~, SY8843QWC:SY8843QWC, F.Cu at (120.1, 118.8)
- added FL1: DLW21SZ900HQ2L, Inductor_SMD:L_CommonModeChoke_Coilcraft_0805USB, F.Cu at (117.1, 104.7)
- added J1: Conn_02x12_Odd_Even, Connector_Hirose:Hirose_DF11-24DP-2DSA_2x12_P2.00mm_Vertical, F.Cu at (135.3, 96.7)
- added J2: Conn_02x12_Odd_Even, Connector_Hirose:Hirose_DF11-24DP-2DSA_2x12_P2.00mm_Vertical, F.Cu at (105.2, 74.8)
- added J3: Conn_01x04, Connector_Molex:Molex_KK-254_AE-6410-04A_1x04_P2.54mm_Vertical, F.Cu at (133.2, 104.0)
- added J4: Conn_02x12_Odd_Even, Connector_Hirose:Hirose_DF11-24DP-2DSA_2x12_P2.00mm_Vertical, F.Cu at (139.1, 68.7)
- added J5: USB_C_Receptacle_USB2.0_14P, Connector_USB:USB_C_Receptacle_GCT_USB4105-xx-A_16P_TopMnt_Horizontal, F.Cu at (107.9, 113.0)
- added L2: VHF160808H33NJT, Inductor_SMD:L_0603_1608Metric, F.Cu at (111.0, 94.5)
- added L4: 0.68uH, Inductor_SMD:L_Cenker_CKCS4020, F.Cu at (116.6, 118.5)
- added R1: 18R, PCM_Resistor_SMD_AKL:R_01005_0402Metric, F.Cu at (112.4, 109.9)
- added R10: 400R, PCM_Resistor_SMD_AKL:R_01005_0402Metric, F.Cu at (104.4, 102.9)
- added R11: 400R, PCM_Resistor_SMD_AKL:R_01005_0402Metric, F.Cu at (104.4, 104.6)
- added R13: 41К, Resistor_SMD:R_0402_1005Metric, F.Cu at (121.5, 116.2)
- added R14: 9.1K, Resistor_SMD:R_0402_1005Metric, F.Cu at (121.5, 118.1)
- added R2: 18R, PCM_Resistor_SMD_AKL:R_01005_0402Metric, F.Cu at (111.9, 109.3)
- added R3: 5.1K, PCM_Resistor_SMD_AKL:R_01005_0402Metric, F.Cu at (114.1, 110.5)
- added R4: 5.1K, PCM_Resistor_SMD_AKL:R_01005_0402Metric, F.Cu at (111.4, 107.8)
- added R5: 10K, Resistor_SMD:R_0402_1005Metric, F.Cu at (120.6, 114.6)
- added R6: 100K, PCM_Resistor_SMD_AKL:R_01005_0402Metric, F.Cu at (158.9, 85.0)
- added R7: 100K, PCM_Resistor_SMD_AKL:R_01005_0402Metric, F.Cu at (126.3, 99.6)
- added R8: 2K, PCM_Resistor_SMD_AKL:R_01005_0402Metric, F.Cu at (159.0, 89.7)
- added R9: 400R, PCM_Resistor_SMD_AKL:R_01005_0402Metric, F.Cu at (104.4, 101.0)
- added SW1: SW_Push, Button_Switch_SMD:SW_SPST_PTS810, F.Cu at (162.2, 85.8)
- added SW2: SW_Push, Button_Switch_SMD:SW_SPST_PTS810, F.Cu at (162.2, 90.6)
- added U2: USBLC6-2SC6, Package_TO_SOT_SMD:SOT-23-6, F.Cu at (114.3, 107.5)
- added Y1: X322512MSB4SI, Crystal:Crystal_SMD_3225-4Pin_3.2x2.5mm, F.Cu at (118.8, 76.9)
- moved L1 11.2 mm to (113.2, 95.8), turned to -90 degrees
- moved U1 4.73 mm to (122.1, 98.0), turned to 180 degrees
- moved DD1 0.80 mm to (119.7, 86.5), turned to 180 degrees
Connections:
- DD1 pad 1: unconnected-(DD1-GPIO4-Pad1) -> IO4
- DD1 pad 10: unconnected-(DD1-DVDD_1-Pad10) -> Net-(DD1-DVDD_1)
- DD1 pad 11: unconnected-(DD1-GPIO12-Pad11) -> IO12
- DD1 pad 12: unconnected-(DD1-GPIO13-Pad12) -> IO13
- DD1 pad 13: unconnected-(DD1-GPIO14-Pad13) -> IO14
- DD1 pad 14: unconnected-(DD1-GPIO15-Pad14) -> IO15
- DD1 pad 15: unconnected-(DD1-IOVDD_2-Pad15) -> +3V3
- DD1 pad 16: unconnected-(DD1-GPIO16-Pad16) -> IO16
- DD1 pad 17: unconnected-(DD1-GPIO17-Pad17) -> IO17
- DD1 pad 18: unconnected-(DD1-GPIO18-Pad18) -> IO18
- DD1 pad 19: unconnected-(DD1-GPIO19-Pad19) -> IO19
- DD1 pad 2: unconnected-(DD1-GPIO5-Pad2) -> IO5
- DD1 pad 20: unconnected-(DD1-GPIO20-Pad20) -> IO20
- DD1 pad 21: unconnected-(DD1-GPIO21-Pad21) -> IO21
- DD1 pad 22: unconnected-(DD1-GPIO22-Pad22) -> IO22
- DD1 pad 23: unconnected-(DD1-GPIO23-Pad23) -> IO23
- DD1 pad 24: unconnected-(DD1-IOVDD_3-Pad24) -> +3V3
- DD1 pad 25: unconnected-(DD1-GPIO24-Pad25) -> IO24
- DD1 pad 26: unconnected-(DD1-GPIO25-Pad26) -> IO25
- DD1 pad 27: unconnected-(DD1-GPIO26-Pad27) -> IO26
- DD1 pad 28: unconnected-(DD1-GPIO27-Pad28) -> IO27
- DD1 pad 29: unconnected-(DD1-IOVDD_4-Pad29) -> +3V3
- DD1 pad 3: unconnected-(DD1-GPIO6-Pad3) -> IO6
- DD1 pad 30: unconnected-(DD1-XIN-Pad30) -> Net-(DD1-XIN)
- DD1 pad 31: unconnected-(DD1-XOUT-Pad31) -> Net-(DD1-XOUT)
- DD1 pad 32: unconnected-(DD1-DVDD_2-Pad32) -> Net-(DD1-DVDD_1)
- DD1 pad 33: unconnected-(DD1-SWCLK-Pad33) -> SWCLK
- DD1 pad 34: unconnected-(DD1-SWDIO-Pad34) -> SWDIO
- DD1 pad 35: unconnected-(DD1-RUN-Pad35) -> RUN
- DD1 pad 36: unconnected-(DD1-GPIO28-Pad36) -> IO28
- DD1 pad 37: unconnected-(DD1-GPIO29-Pad37) -> IO29
- DD1 pad 38: unconnected-(DD1-GPIO30-Pad38) -> IO30
- DD1 pad 39: unconnected-(DD1-GPIO31-Pad39) -> IO31
- DD1 pad 4: unconnected-(DD1-GPIO7-Pad4) -> IO7
- DD1 pad 40: unconnected-(DD1-GPIO32-Pad40) -> IO32
- DD1 pad 41: unconnected-(DD1-IOVDD_5-Pad41) -> +3V3
- DD1 pad 42: unconnected-(DD1-GPIO33-Pad42) -> IO33
- DD1 pad 43: unconnected-(DD1-GPIO34-Pad43) -> IO34
- DD1 pad 44: unconnected-(DD1-GPIO35-Pad44) -> IO35
- DD1 pad 45: unconnected-(DD1-GPIO36-Pad45) -> IO36
- DD1 pad 46: unconnected-(DD1-GPIO37-Pad46) -> IO37
- DD1 pad 47: unconnected-(DD1-GPIO38-Pad47) -> IO38
- DD1 pad 48: unconnected-(DD1-GPIO39-Pad48) -> IO39
- DD1 pad 49: unconnected-(DD1-GPIO40_ADC0-Pad49) -> IO40
- DD1 pad 5: unconnected-(DD1-IOVDD_1-Pad5) -> +3V3
- DD1 pad 50: unconnected-(DD1-IOVDD_6-Pad50) -> +3V3
- DD1 pad 51: unconnected-(DD1-DVDD_3-Pad51) -> Net-(DD1-DVDD_1)
- DD1 pad 52: unconnected-(DD1-GPIO41_ADC1-Pad52) -> IO41
- DD1 pad 53: unconnected-(DD1-GPIO42_ADC2-Pad53) -> IO42
- DD1 pad 54: unconnected-(DD1-GPIO43_ADC3-Pad54) -> IO43
- DD1 pad 55: unconnected-(DD1-GPIO44_ADC4-Pad55) -> IO44
- DD1 pad 56: unconnected-(DD1-GPIO45_ADC5-Pad56) -> IO45
- DD1 pad 57: unconnected-(DD1-GPIO46_ADC6-Pad57) -> IO46
- DD1 pad 58: unconnected-(DD1-GPIO47_ADC7-Pad58) -> IO47
- DD1 pad 59: unconnected-(DD1-ADC_AVDD-Pad59) -> Net-(DD1-ADC_AVDD)
- DD1 pad 6: unconnected-(DD1-GPIO8-Pad6) -> IO8
- DD1 pad 60: unconnected-(DD1-IOVDD_7-Pad60) -> +3V3
- DD1 pad 61: unconnected-(DD1-VREG_AVDD-Pad61) -> Net-(DD1-ADC_AVDD)
- DD1 pad 62: unconnected-(DD1-VREG_PGND-Pad62) -> Earth
- DD1 pad 63: unconnected-(DD1-VREG_LX-Pad63) -> Net-(DD1-VREG_LX)
- DD1 pad 64: unconnected-(DD1-VREG_VIN-Pad64) -> +3V3
- DD1 pad 65: unconnected-(DD1-VREG_FB-Pad65) -> Net-(DD1-DVDD_1)
- DD1 pad 66: unconnected-(DD1-USB_DM-Pad66) -> USB_mcu-
- DD1 pad 67: unconnected-(DD1-USB_DP-Pad67) -> USB_mcu+
- DD1 pad 68: unconnected-(DD1-USB_OTP_VDD-Pad68) -> +3V3
- DD1 pad 69: unconnected-(DD1-QSPI_IOVDD-Pad69) -> +3V3
- DD1 pad 7: unconnected-(DD1-GPIO9-Pad7) -> IO9
- DD1 pad 70: unconnected-(DD1-QSPI_SD3-Pad70) -> QSPI_SD3
- DD1 pad 71: unconnected-(DD1-QSPI_SCLK-Pad71) -> QSPI_CLK
- DD1 pad 72: unconnected-(DD1-QSPI_SD0-Pad72) -> QSPI_SD0
- DD1 pad 73: unconnected-(DD1-QSPI_SD2-Pad73) -> QSPI_SD2
- DD1 pad 74: unconnected-(DD1-QSPI_SD1-Pad74) -> QSPI_SD1
- DD1 pad 75: unconnected-(DD1-QSPI_SS-Pad75) -> QSPI_SS
- DD1 pad 76: unconnected-(DD1-IOVDD_8-Pad76) -> +3V3
- DD1 pad 77: unconnected-(DD1-GPIO0-Pad77) -> IO0
- DD1 pad 78: unconnected-(DD1-GPIO1-Pad78) -> IO1
- DD1 pad 79: unconnected-(DD1-GPIO2-Pad79) -> IO2
- DD1 pad 8: unconnected-(DD1-GPIO10-Pad8) -> IO10
- DD1 pad 80: unconnected-(DD1-GPIO3-Pad80) -> IO3
- DD1 pad 81: unconnected-(DD1-GND-Pad81) -> Earth
- DD1 pad 9: unconnected-(DD1-GPIO11-Pad9) -> IO11
- L1 pad 1: unconnected-(L1-Pad1) -> Net-(DD1-VREG_LX)
- L1 pad 2: unconnected-(L1-Pad2) -> Net-(DD1-DVDD_1)
- U1 pad 1: unconnected-(U1-~{CS}-Pad1) -> QSPI_SS
- U1 pad 2: unconnected-(U1-DO/IO_{1}-Pad2) -> QSPI_SD1
- U1 pad 3: unconnected-(U1-~{WP}/IO_{2}-Pad3) -> QSPI_SD2
- U1 pad 4: unconnected-(U1-GND-Pad4) -> Earth
- U1 pad 5: unconnected-(U1-DI/IO_{0}-Pad5) -> QSPI_SD0
- U1 pad 6: unconnected-(U1-CLK-Pad6) -> QSPI_CLK
- U1 pad 7: unconnected-(U1-~{HOLD}/~{RESET}/IO_{3}-Pad7) -> QSPI_SD3
- U1 pad 8: unconnected-(U1-VCC-Pad8) -> +3V3
- U1 pad 9: unconnected-(U1-EP-Pad9) -> Earth
Routing:
- net +3V3: track 0.00 -> 192.6 mm, vias 0 -> 30
- net IO9: track 0.00 -> 91.8 mm, vias 0 -> 1
- net QSPI_SS: track 0.00 -> 52.9 mm
- net RUN: track 0.00 -> 52.8 mm, vias 0 -> 2
- net Net-(DD1-DVDD_1): track 0.00 -> 42.9 mm, vias 0 -> 5
- net SWDIO: track 0.00 -> 31.9 mm, vias 0 -> 1
- net SWCLK: track 0.00 -> 30.6 mm, vias 0 -> 1
- net IO27: track 0.00 -> 29.3 mm
- net IO25: track 0.00 -> 29.2 mm
- net IO26: track 0.00 -> 27.2 mm
- net IO24: track 0.00 -> 27.0 mm
- net VCC-5V: track 0.00 -> 18.7 mm, vias 0 -> 35
- net IO23: track 0.00 -> 18.5 mm
- net IO1: track 0.00 -> 17.4 mm
- net IO47: track 0.00 -> 17.1 mm
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- added copper zone on B.Cu, net +3V3
- added copper zone on F.Cu, net +3V3
- added copper zone on B.Cu, net Earth
- added copper zone on F.Cu, net Earth
- added copper zone on F.Cu, net Net-(DD5-LX)
- added copper zone on B.Cu, net VCC-5V
- added copper zone on F.Cu, net VCC-5V

Commit message: Закончил :)
Parts:
- added G***: LOGO, LOGO, F.Cu at (148.1, 85.3)
- added G***: LOGO, LOGO, F.Cu at (142.1, 118.3)
- added G***: LOGO, LOGO, B.Cu at (120.0, 89.9)
- added G***: LOGO, LOGO, B.Cu at (140.4, 115.0)
- added kibuzzard-67ED7B45: G***, kibuzzard-67ED7B45, F.Cu at (136.4, 114.4)
Other:
- board text added: "BOOT"
- board text added: "RST"
- board text added: "by @madjogger"
- board text added: "dev board"
